File: raspi-hat/raspi-adapter.brd (EAGLE design)
At the start: 56.5 x 65.1 mm, 37 parts, among them IC1 24C01SN, Q1 BSS138

Commit message: review schematic and layout
Parts:
- removed JP12, JP15, JP9: (no value), SparkFun-Passives:1X02
- removed JP13: (no value), adafruit:1X03
- removed L1, L2, L3, L4: WS2812B, adafruit:WS2812B
- removed SW3, SW4: (no value), adafruit:PUSHBUTTON_SMD_SJ
- added SW1, SW2: (no value), adafruit:PUSHBUTTON_SMD_SJ
- added X10, X11, X2: (no value), adafruit:1X03
- added X4: (no value), adafruit:1X08-CLEANBIG
- added X8: (no value), adafruit:1X06-BIG
- added X9: HAT-Conn, adafruit:2X20
- C1: value 1u -> 100u; device rcl:C0603 -> rcl:C1210
- C2: value 10n -> 1u
- C3: value 100u -> 10n; device rcl:C1210 -> rcl:C0603
- JP1: value HAT-Conn -> (none); device adafruit:2X20 -> SparkFun-Passives:1X02
- JP2: device adafruit:1X08-CLEANBIG -> SparkFun-Passives:1X02
- JP3: device adafruit:1X06-BIG -> SparkFun-Passives:1X02
- JP5: device adafruit:1X03 -> SparkFun-Passives:1X02
- R2: value 3k9 -> 270
- R5: value 270 -> 3k9
- moved JP5 61.0 mm to (50.8, 62.2), turned to 270 degrees
- moved JP3 58.4 mm to (53.7, 14.3), turned to 270 degrees
- moved JP2 53.4 mm to (35.6, 1.27), turned to 90 degrees
- moved JP6 44.5 mm to (48.3, 59.7), turned to 90 degrees
- moved JP7 36.2 mm to (53.7, 16.8), turned to 90 degrees
- moved R2 34.1 mm to (21.6, 14.0)
- moved JP1 33.5 mm to (40.0, 3.81)
- moved R5 28.6 mm to (53.3, 26.4), turned to 180 degrees
- moved C3 24.1 mm to (41.6, 14.0)
- moved V+NEO 22.9 mm to (16.2, 2.54)
- moved V-NEO 22.9 mm to (23.8, 2.54)
- moved DIN_NEO 22.9 mm to (20.0, 2.54)
- moved C2 22.2 mm to (19.1, 14.9), turned to 90 degrees
- moved JP4 10.3 mm to (17.1, 22.5)
- moved R4 9.94 mm to (53.0, 23.5), turned to 90 degrees
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- renumbered JP10 to X6, JP11 to X7, JP14 to X1, JP8 to X3, U$3 to X5
Connections:
- removed net N$1: L2.2, L3.4
- removed net N$3: L3.2, L4.4
- removed net N$5: L1.4, Q1.3, R5.1
- removed net N$9: JP4.1, VEXT+.1
- new net +5V: C1.1, R2.2, V+NEO.1, X2.2
- new net 3V3_RPI: JP2.2, X9.1, X9.17
- new net VIN_RPI: JP1.2, X9.2, X9.4
- net +3V3: now also C3.1, JP2.1, R5.2, SW2.P$1; no longer C2.1, JP1.1, JP1.17, R2.2, SW4.P$1
- net GND: now also SW1.P$1, X11.1, X11.2, X11.3, X8.1, X9.14, X9.20, X9.25, X9.30, X9.34, X9.39, X9.6, X9.9; no longer JP1.14, JP1.20, JP1.25, JP1.30, JP1.34, JP1.39, JP1.6, JP1.9, JP13.1, JP13.2, JP13.3, JP3.1, L1.3, L2.3, L3.3, L4.3, SW3.P$1
- net LED_BLUE: now also X10.1, X9.35; no longer JP1.35, JP5.1
- net LED_GREEN: now also X10.3, X9.40; no longer JP1.40, JP5.3
- net LED_RED: now also X9.15; no longer JP1.15
- net LED_YELLOW: now also X10.2, X9.38; no longer JP1.38, JP5.2
- net N$2: now also VEXT+.1, X2.1; no longer L1.2, L2.4
- net N$4: now also SW2.P$2; no longer SW4.P$2
- net N$6: now also Q1.3, R2.1; no longer L4.2
- net N$7: now also JP4.1, X9.16; no longer JP1.16, JP7.1
- net RST: now also JP4.2, SW1.P$2; no longer JP7.2, SW3.P$2
- net SCL: now also JP3.2, R4.1; no longer JP6.2, R3.1
- net SDA: now also JP7.1, R5.1; no longer JP15.1, R2.1
- net V+: now also C2.1, JP1.1, X2.3; no longer C1.1, C3.1, JP1.2, JP1.4, JP4.2, L1.1, L2.1, L3.1, L4.1, R5.2, V+NEO.1
- net X1: now also JP5.1, X4.8, X9.5; no longer JP1.5, JP12.1, JP2.8
- net X1_: now also JP5.2, X9.8; no longer JP1.8, JP12.2
- net X2: now also JP6.1, X4.7, X9.3; no longer JP1.3, JP2.7, JP9.1
- net X2_2: now also JP6.2, X9.10; no longer JP1.10, JP9.2
- net X3: now also X4.6, X9.11; no longer JP1.11, JP2.6
- net X4: now also X4.5, X9.13; no longer JP1.13, JP2.5
- net X5: now also R3.1, X4.4; no longer JP2.4, R4.1
- net X6: now also X4.3; no longer JP2.3
- net X7: now also X4.2; no longer JP2.2
- net X8: now also X4.1; no longer JP2.1
- net Y1: now also X8.5; no longer JP3.5
- net Y10: now also JP7.2, X9.27; no longer JP1.27, JP15.2
- net Y2: now also X8.4; no longer JP3.4
- net Y3: now also X9.12; no longer JP1.12
- net Y4: now also X9.7; no longer JP1.7
- net Y5: now also X9.24; no longer JP1.24
- net Y6: now also X9.23; no longer JP1.23
- net Y7: now also X9.21; no longer JP1.21
- net Y8: now also X9.19; no longer JP1.19
- net Y9: now also JP3.1, X9.28; no longer JP1.28, JP6.1
Routing:
- net V+: track 116.7 -> 54.5 mm, vias 12 -> 5
- net GND: track 76.7 -> 38.7 mm, vias 11 -> 19
- net N$5: track 26.5 -> 0.00 mm, vias 2 -> 0
- net +5V: track 0.00 -> 17.8 mm
- net +3V3: track 37.1 -> 49.0 mm, vias 6 -> 9
- net N$1: track 8.20 -> 0.00 mm, vias 2 -> 0
- net N$3: track 8.20 -> 0.00 mm, vias 2 -> 0
- net N$6: track 11.6 -> 17.5 mm
- net N$9: track 5.79 -> 0.00 mm
- net SCL: track 24.3 -> 21.3 mm
- net X8: track 55.8 -> 58.8 mm
- net RST: track 55.5 -> 52.8 mm
- net VIN_RPI: track 0.00 -> 2.54 mm
- net X1_: track 18.1 -> 16.2 mm
- net VIN: track 19.7 -> 18.1 mm
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- added copper zone on layer 1, net +3V3
- added copper zone on layer 15, net 3V3_RPI
- added copper zone on layer 15, net VIN_RPI
Other:
- board text added: "3V3"
- board text added: "5V"
- board text added: "HAT-EE"
- board text added: "Int"
- board text added: "RE"
- board text added: "Raspi/HAT"
- board text removed: "Neopixels"
- board text removed: "Raspberry/HAT"

Commit message: working in review, removed onboard neopixel
Parts:
- removed R3: 3k9, resistor:R0603
- removed X1: (no value), adafruit:1X03
- added JP8: (no value), SparkFun-Passives:1X02
- C1: device rcl:C1210 -> rcl:C2220K
- JP1: device SparkFun-Passives:1X02 -> adafruit:1X01
- V+: value V+NEO -> V+
- moved JP2 57.8 mm to (34.9, 59.1), turned to 0 degrees
- moved JP1 27.3 mm to (19.1, 21.3), turned to 0 degrees
- moved SW1 17.2 mm to (32.7, 3.17)
- moved SW2 11.5 mm to (41.6, 3.17)
- moved R1 5.24 mm to (25.7, 19.1), turned to 0 degrees
- moved R2 5.02 mm to (25.7, 16.8), turned to 0 degrees
- moved C1 2.29 mm to (24.1, 11.4)
- moved JP5 1.42 mm to (52.1, 61.6)
- moved JP6 1.42 mm to (49.5, 59.1)
- moved JP4 1.42 mm to (16.5, 21.3)
- moved X8 0.71 mm to (20.0, 61.6)
- moved R4 0.64 mm to (53.0, 22.9)
- moved R5 0.45 mm to (53.0, 26.0), turned to 270 degrees
- renumbered DIN_NEO to CLK_OUT, V+NEO to V+, V-NEO to V-
Connections:
- removed net VIN_RPI: JP1.2, X9.2, X9.4
- net +3V3: no longer R3.2
- net GND: now also IC1.7; no longer X1.2
- net LED_RED: no longer X9.15
- net V+: now also X9.2, X9.4; no longer JP1.1
- net X1: no longer X9.5
- net X10: now also X9.3
- net X11: now also X9.26
- net X12: now also X9.22
- net X2: no longer X9.3
- net X5: now also X9.18; no longer IC1.7, R3.1
- net X9: now also X9.5
- net Y10: now also JP8.2; no longer X1.3
- net Y11: now also X9.15
- net Y12: now also JP1.1
- net Y9: now also JP8.1; no longer X1.1
Routing:
- net Y11: track 0.00 -> 67.8 mm, vias 0 -> 1
- net X9: track 0.00 -> 60.8 mm, vias 0 -> 1
- net X10: track 0.00 -> 56.5 mm, vias 0 -> 1
- net 3V3_RPI: track 0.00 -> 43.2 mm
- net X11: track 0.00 -> 34.5 mm, vias 0 -> 1
- net Y12: track 0.00 -> 34.0 mm
- net X12: track 0.00 -> 25.9 mm, vias 0 -> 1
- net +3V3: track 49.0 -> 27.6 mm, vias 9 -> 6
- net RST: track 52.8 -> 71.4 mm
- net N$4: track 20.9 -> 38.4 mm
- net LED_RED: track 14.2 -> 0.00 mm
- net X1: track 28.0 -> 15.2 mm, vias 0 -> 1
- net X5: track 57.6 -> 69.8 mm, vias 0 -> 2
- net V+: track 54.5 -> 44.7 mm, vias 5 -> 1
- net GND: track 38.7 -> 48.3 mm
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- removed copper zone on layer 15, net 3V3_RPI
- removed copper zone on layer 15, net VIN_RPI
Other:
- board text added: "1"
- board text added: "11"
- board text added: "21"
- board text added: "GP"
- board text added: "I2C"
- board text added: "RP"
- board text removed: "5V"
- board text removed: "I2C2"
- board text removed: "RPi"
